Commit message: quadlrotorをarm_kinnikuに変更

File: robots/arm_kinniku/urdf/robot.gazebo.xacro (robot description, xacro)
@@ -1,8 +1,8 @@
 <?xml version="1.0"?>
 <robot
-    xmlns:xacro="http://www.ros.org/wiki/xacro" name="mini_quadrotor" >
-  <xacro:arg name="robot_name" default="quadrotor" />
+    xmlns:xacro="http://www.ros.org/wiki/xacro" name="arm_kinniku" >
+  <xacro:arg name="robot_name" default="arm_kinniku" />
   <!-- robot urdf -->
-  <xacro:include filename="$(find mini_quadrotor)/urdf/robot.urdf.xacro" />
+  <xacro:include filename="$(find arm_kinniku)/urdf/robot.urdf.xacro" />
   <!-- gazebo plugin for default controller and sensors -->
   <xacro:include filename="$(find aerial_robot_simulation)/xacro/spinal.gazebo.xacro" />

File: robots/arm_kinniku/urdf/robot.urdf.xacro (robot description, xacro)
@@ -1,5 +1,5 @@
 <?xml version="1.0"?>
 <robot
-    xmlns:xacro="http://www.ros.org/wiki/xacro" name="module_quadrotor" >
+    xmlns:xacro="http://www.ros.org/wiki/xacro" name="arm_kinniku" >
   <!-- general attribute -->
   <baselink name="fc" />
@@ -58,5 +58,5 @@
         <origin rpy="0 0 0" xyz="0 0 0"/>
         <geometry>
-          <mesh filename="package://mini_quadrotor/urdf/mesh/prop_5inch.dae" />
+          <mesh filename="package://arm_kinniku/urdf/mesh/prop_5inch.dae" />
         </geometry>
       </visual>
@@ -106,5 +106,5 @@
       <origin rpy="0 0 0" xyz="0 0 0"/>
       <geometry>
-        <mesh filename="package://mini_quadrotor/urdf/mesh/main_body_livox.dae" />
+        <mesh filename="package://arm_kinniku/urdf/mesh/main_body_livox.dae" />
       </geometry>
     </visual>
@@ -149,5 +149,5 @@
   </xacro:extra_module>
   <!-- battery -->
-  <xacro:extra_module name = "battery" parent = "main_body" visible = "1" model_url = "package://mini_quadrotor/urdf/mesh/turnigy_3S_2200mAh.dae" >
+  <xacro:extra_module name = "battery" parent = "main_body" visible = "1" model_url = "package://arm_kinniku/urdf/mesh/turnigy_3S_2200mAh.dae" >
     <origin xyz="0.0 0 -0.035" rpy="${pi/2} 0 0"/>
     <inertial>
